Commit message: urdf_gazebo

File: nebulizador_description/robot/urdf/arm.urdf.xacro (robot description, xacro)
@@ -33,9 +33,9 @@
         <parent link="box_nebulizador"/>
         <child link="box_nebulizador_base"/>
-        <origin xyz="0.0 0.0 0.3825" rpy="0.0 0.0 0.0" />
+        <origin xyz="0.0 0.0 0.3825" rpy="0.0 0.0 3.14159" />
     </joint>
     <xacro:joint_v1 joint_name="J1"
                   parent_name="box_nebulizador_base" child_name="link_1"
-                  ox="0" oy="0" oz="0.017"
+                  ox="-0.16" oy="0" oz="0.017"
                   roll="0" pitch="0" yaw="-1.5708"
                   ax="0" ay="0" az="1"

File: nebulizador_description/urdf/accessories/arm/body.urdf.xacro (robot description, xacro)
@@ -9,4 +9,5 @@
           <mesh filename="package://nebulizador_description/meshes/arm/visual/${name}.stl" scale="0.001 0.001 0.001"/>
         </geometry>
+        <material name="grey"/>
       </visual>
       <!--collision>

File: nebulizador_description/urdf/accessories/box.urdf.xacro (robot description, xacro)
@@ -4,8 +4,8 @@
         <visual>
             <geometry>
-                <box size="0.515487 0.233457 0.765"/>
+                <box size="0.515487 0.233457 0.78"/>
                 <!--mesh filename="package://nebulizador_description/meshes/arm/visual/base_link.stl" scale="0.001 0.001 0.001"/-->
             </geometry>
-            <material name="white"/>
+            <material name="black"/>
         </visual>
     </link>
@@ -13,5 +13,5 @@
         <parent link="mount_point_link"/>
         <child link="box_nebulizador"/>
-        <origin xyz="0.0 0.0 0.06"/>
+        <origin xyz="0.0 0.0 0.0"/>
     </joint>
 </robot>
